Commit message: new robot xacro

File: description/robot_core.xacro (robot description, xacro)
@@ -2,14 +2,14 @@
 <robot xmlns:xacro="http://www.ros.org/wiki/xacro" >
     <xacro:include filename="inertial_macros.xacro"/>
-    <xacro:property name="chassis_length" value="0.26"/>
-    <xacro:property name="chassis_width" value="0.15"/>
-    <xacro:property name="chassis_height" value="0.065"/>
+    <xacro:property name="chassis_length" value="0.3"/>
+    <xacro:property name="chassis_width" value="0.3"/>
+    <xacro:property name="chassis_height" value="0.15"/>
     <xacro:property name="chassis_mass" value="0.5"/>
     <xacro:property name="wheel_radius" value="0.0325"/>
     <xacro:property name="wheel_thickness" value="0.026"/>
     <xacro:property name="wheel_mass" value="0.05"/>
-    <xacro:property name="wheel_offset_x" value="0.055"/>
-    <xacro:property name="wheel_offset_y" value="0.0625"/>
-    <xacro:property name="wheel_offset_z" value="-0.0225"/>
+    <xacro:property name="wheel_offset_x" value="0.085"/>
+    <xacro:property name="wheel_offset_y" value="0.17"/>
+    <xacro:property name="wheel_offset_z" value="-0.0625"/>
     <material name="white"> <color rgba="1 1 1 1" /> </material>
     <material name="orange"> <color rgba="1 0.3 0.1 1"/> </material>
@@ -63,7 +63,13 @@
         </link>
         <gazebo reference="${prefix}_${side}_wheel">
-            <material>Gazebo/Red</material>
-            <mu1>1.0</mu1>
-            <mu2>0.2</mu2>
+            <material>Gazebo/Yellow</material>
+            <xacro:if value="${prefix == 'front'}"> <!-- Apply normal friction to FRONT wheels -->
+                <mu1>1.0</mu1>
+                <mu2>0.2</mu2> <!-- Allow some sideways slip for steering if needed -->
+            </xacro:if>
+            <xacro:if value="${prefix == 'rear'}">  <!-- Apply very low friction to REAR wheels -->
+                <mu1>0.001</mu1> <!-- Minimal forward/backward friction -->
+                <mu2>0.001</mu2> <!-- Minimal sideways friction -->
+            </xacro:if>
         </gazebo>
     </xacro:macro>
